File: KiCAD Layout/KiCAD Layout.kicad_sch (KiCad schematic)
At the start: 4 parts

Commit message: Updated KiCAD
Connections:
- net at U1. (VCC): now also U3. (VCC)
- net at U3. (VCC): no longer U1. (VCC)
- net at U4. (VCC): now also U2. (VCC)
- new net: U1. (VCC), U3. (VCC) (x9)
- new net: U2. (VCC), U4. (VCC) (x9)
- now unconnected: U3. (VCC), U3. (VCC), U3. (VCC), U3. (VCC), U3. (VCC), U3. (VCC), U3. (VCC), U3. (VCC), U3. (VCC)
- no-connect marks 0 -> 4

Commit message: Updates to KiCAD
Parts:
- added U5: WeMos_D1_mini, Module:WEMOS_D1_mini_light, symbol MCU_Module:WeMos_D1_mini
- added U6: ~, symbol New_Library:Arduino_Mega
- added U7: ~, symbol New_Library:Level_Shifter
Connections:
- net at U1. (VCC): now also U3. (VCC)
- net at U3. (VCC): no longer U1. (VCC)
- net at U4. (VCC): now also U2. (VCC)
- net at U2. (VCC): no longer U4. (VCC)
- new net: U1. (VCC), U3. (VCC) (x9)
- new net: U2. (VCC), U4. (VCC) (x9)
- now unconnected: U2. (VCC), U2. (VCC), U2. (VCC), U2. (VCC), U2. (VCC), U2. (VCC), U2. (VCC), U2. (VCC), U2. (VCC), U3. (VCC), U3. (VCC), U3. (VCC), U3. (VCC), U3. (VCC), U3. (VCC), U3. (VCC), U3. (VCC), U3. (VCC)
